File: Lumen-Driver-X2.sch (EAGLE design)
At the start: 30 parts, among them J1 AVR_SPI_PRG_6PTH, U1 Tiny45-20-SMT, Y1 8Mhz

Commit message: Updated R2 design. Ordered and tested.
Parts:
- removed C2: 0.68uF 100V, resistor:C-EUC0805
- removed U$10: LOGOBR-LOGO-MS-COPPER, BlueRobotics-Main:LOGOBR-LOGO-MS-COPPER
- removed U$2: LED-MK-R, BlueRobotics-Main:LED-MK-R
Connections:
- removed net EXT: U$2.THERMAL
- removed net LED+ISO: C2.2, U$2.A
- removed net LED-ISO: C2.1, U$2.C
Other:
- note removed: "MKRAWT-00-0000-0B00H4051"
