File: Lumen.brd (EAGLE design)
At the start: 59.3 x 24 mm, 30 parts, among them J1 AVR_SPI, U1 Tiny45-20-SMT, Y1 8Mhz

Commit message: Minor updates.
Parts:
- C5: value 0.1uF -> 0.1uF 100V; device resistor:C0603 -> resistor:C0805
- moved C5 0.36 mm to (52.0, 11.8)
Other:
- board text removed: "rev5"
Changed lines of the file:
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@@
 <text x="4.125" y="11.25" size="1.27" layer="21" font="vector" rot="SR270" align="center">Lumen Subsea
 Light</text>
-<text x="14.125" y="3.625" size="1.27" layer="21" font="vector" rot="R270" align="center">rev5</text>
+<text x="14.125" y="3.625" size="1.27" layer="21" font="vector" rot="R270" align="center">rev6</text>
 <text x="18.75" y="18.75" size="1.27" layer="21" font="vector" rot="SR270" align="center-left">Blue Robotics</text>
 <polygon width="0.254" layer="29">
@@
 </element>
 <element name="C4" library="resistor" package="C1210" value="4.7uF 80V" x="40.2" y="18.8" rot="R90"/>
-<element name="C5" library="resistor" package="C0603" value="0.1uF" x="52.25" y="11.5" rot="R180"/>
+<element name="C5" library="resistor" package="C0805" value="0.1uF 100V" x="52.05" y="11.8" rot="R180"/>
 <element name="D1" library="BlueRobotics-Main" package="SMA" value="60V 3A" x="45.11" y="15.99" rot="R180"/>
 <element name="J1" library="SparkFun-Connectors" package="2X3" value="AVR_SPI" x="31.69" y="2.5775" smashed="yes" rot="R90">
@@
 <contactref element="C5" pad="2"/>
 <wire x1="48.84" y1="11.38" x2="51.28" y2="11.38" width="0.4064" layer="1"/>
-<wire x1="51.28" y1="11.38" x2="51.4" y2="11.5" width="0.4064" layer="1"/>
+<wire x1="51.28" y1="11.38" x2="51.1" y2="11.8" width="0.4064" layer="1"/>
 </signal>
 <signal name="N$5">
@@
 <vertex x="53.5" y="11.25"/>
 <vertex x="53.5" y="12.25"/>
-<vertex x="52.5" y="12.25"/>
-<vertex x="52.5" y="21.5"/>
+<vertex x="52.8" y="12.25"/>
+<vertex x="52.8" y="21.5"/>
 <vertex x="48.75" y="21.5"/>
 <vertex x="45.5" y="16"/>
@@
 <contactref element="C2" pad="1"/>
 <polygon width="0.4064" layer="1" isolate="0.254" thermals="no">
-<vertex x="53.25" y="25"/>
+<vertex x="53.55" y="25"/>
 <vertex x="59.25" y="25"/>
 <vertex x="59.25" y="20"/>
@@
 <vertex x="54.25" y="10.5"/>
 <vertex x="54.25" y="13"/>
-<vertex x="53.25" y="13"/>
+<vertex x="53.55" y="13"/>
 </polygon>
 <polygon width="0.4064" layer="16" isolate="0.254" thermals="no">
